File: schematics/breakout.kicad_pcb (KiCad board)
At the start: 2 copper layers, 27.3 x 54 mm, 14 parts, among them P1 RPI_HEADER, P2 CONN_01X03, P3 CONN_01X03, P4 CONN_01X03, P5 CONN_01X03, P6 BARREL_JACK, P7 CONN_01X04, P8 CONN_01X04, Q1 BSS138, Q2 BSS138

Commit message: Updated layouts for order
Parts:
- moved C1 1.27 mm to (133.3, 72.4)
- moved C2 1.27 mm to (133.3, 80.0)
- moved C3 1.27 mm to (133.3, 87.6)
- moved C4 1.27 mm to (133.3, 95.2)
Routing:
- net GND: track 159.0 -> 40.3 mm
- net VCC: track 108.8 -> 94.5 mm
Other:
- board size 27.3 x 54 mm -> 26.7 x 54 mm
- net class Default: clearance 0.1524 -> 0.254
- net class Power: clearance 0.1524 -> 0.254
- rule trace_clearance: 0.1524 -> 0.254
- board text removed: "Move caps away from connector"
